File: hardware/mystat_circuit_board/kicad_files/mystat.kicad_pcb (KiCad board)
At the start: 4 copper layers, 60 x 81 mm, 93 parts, among them J1 PJ-063AH, J2 2173157-3, J3 SJ1-42534-SMT, K1 9011-05-11, K2 9011-05-11, K3 9011-05-11, K4 9011-05-11, K5 9011-05-11, P1 ICSP, U10 OPA192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

Commit message: update to KiCAD 10
Other:
- net class Default removed
