File: hardware/mystat_circuit_board/kicad_files/mystat.kicad_pcb (KiCad board)
At the start: 4 copper layers, 60 x 81 mm, 93 parts, among them J1 PJ-063AH, J2 2173157-3, J3 SJ1-42534-SMT-TR, K1 9011-05-11, K2 9011-05-11, K3 9011-05-11, K4 9011-05-11, K5 9011-05-11, P1 ICSP, U10 OPA192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

Commit message: revert to KiCAD 10 state before attempting reed relay changes, to merge into master
Parts:
- C10, C11, C12, C13, C14, C15, C17, C18, C2, C23, C25, C26, C27, C28, C29, C30, C31, C32, C34, C35, C36, C37: value 100 nF -> 0.1 µF
- C16: value 10 uF -> 10 µF
- C24: value 4.7 nF -> 4700 pF
- C3: value 47 uF -> 47 μF
- C39, C5, C6, C8, C9: value 4.7 uF -> 4.7 µF
- C4, C7: value 4.7 uF -> 4.7 μF
- FB1: value 32 Ω -> Ferrite_Bead
- J3: value SJ1-42534-SMT-TR -> SJ1-42534-SMT
- U7, U8: value MCP3551 -> MCP3550-60
Connections:
- J2 pad 4: unconnected-(J2-Pad4) -> (no net)
- P1 pad 6: unconnected-(P1-Pin_6-Pad6) -> (no net)
- U11 pad 1: unconnected-(U11-BW-Pad1) -> (no net)
- U12 pad 5: unconnected-(U12-NC-Pad5) -> (no net)
- U2 pad E1: unconnected-(U2-PIN_E1-PadE1) -> (no net)
- U2 pad F1: unconnected-(U2-PIN_F1-PadF1) -> (no net)
- U5 pad 14: unconnected-(U5-RC2-Pad14) -> (no net)
- U6 pad 1: unconnected-(U6-TP-Pad1) -> (no net)
- U6 pad 3: unconnected-(U6-NIC-Pad3) -> (no net)
- U6 pad 5: unconnected-(U6-TRIM-Pad5) -> (no net)
- U6 pad 7: unconnected-(U6-NIC-Pad7) -> (no net)
- U6 pad 8: unconnected-(U6-TP-Pad8) -> (no net)
- U9 pad 6: unconnected-(U9-DNC-Pad6) -> (no net)
- U9 pad 7: unconnected-(U9-DNC-Pad7) -> (no net)
- U9 pad 8: unconnected-(U9-DNC-Pad8) -> (no net)

Commit message: merged Daniel's changes in to GUI. getting things ready in KiCAD 10 and finding substitute parts
Parts:
- C10, C11, C12, C13, C14, C15, C17, C18, C2, C23, C25, C26, C27, C28, C29, C30, C31, C32, C34, C35, C36, C37: value 0.1 µF -> 100 nF
- C16: value 10 µF -> 10 uF
- C24: value 4700 pF -> 4.7 nF
- C3: value 47 μF -> 47 uF
- C39, C5, C6, C8, C9: value 4.7 µF -> 4.7 uF
- C4, C7: value 4.7 μF -> 4.7 uF
- FB1: value Ferrite_Bead -> 32 Ω
- J3: value SJ1-42534-SMT -> SJ1-42534-SMT-TR
- U7, U8: value MCP3550-60 -> MCP3551
Connections:
- J2 pad 4: (no net) -> unconnected-(J2-Pad4)
- P1 pad 6: (no net) -> unconnected-(P1-Pin_6-Pad6)
- U11 pad 1: (no net) -> unconnected-(U11-BW-Pad1)
- U12 pad 5: (no net) -> unconnected-(U12-NC-Pad5)
- U2 pad E1: (no net) -> unconnected-(U2-PIN_E1-PadE1)
- U2 pad F1: (no net) -> unconnected-(U2-PIN_F1-PadF1)
- U5 pad 14: (no net) -> unconnected-(U5-RC2-Pad14)
- U6 pad 1: (no net) -> unconnected-(U6-TP-Pad1)
- U6 pad 3: (no net) -> unconnected-(U6-NIC-Pad3)
- U6 pad 5: (no net) -> unconnected-(U6-TRIM-Pad5)
- U6 pad 7: (no net) -> unconnected-(U6-NIC-Pad7)
- U6 pad 8: (no net) -> unconnected-(U6-TP-Pad8)
- U9 pad 6: (no net) -> unconnected-(U9-DNC-Pad6)
- U9 pad 7: (no net) -> unconnected-(U9-DNC-Pad7)
- U9 pad 8: (no net) -> unconnected-(U9-DNC-Pad8)
