File: hardware/mystat_circuit_board/kicad_files/mystat.kicad_pcb (KiCad board)
At the start: 4 copper layers, 60 x 81 mm, 93 parts, among them J1 PJ-063AH, J4 Screw_Terminal_01x04, P1 ICSP, U10 OPA192, U11 BUF634AIDDAR, U12 ADG1419, U13 OPA192, U14 OPA192, U15 OPA192, U16 OPA192, U17 OPA192, U2 LTM8045, U3 ADP7182AUJZ-R7, U4 ADP7118AUJZ-5.0-R7, U5 PIC16F1459, U6 ADR421, U7 MCP3551, U8 MCP3551, U9 DAC1220, X1 2.5 MHz

Commit message: mostly resistor changes
Parts:
- C16: footprint Capacitor_SMD:C_1210_3225Metric -> Capacitor_SMD:C_0805_2012Metric
- C19, C20, C33, C38: footprint Capacitor_SMD:C_0805_2012Metric -> Capacitor_SMD:C_0603_1608Metric
- C24: value 4700 pF -> 4.7 nF
- C3: footprint easyeda2kicad:CAP-SMD_BD5.0-L5.3-W5.3-LS6.0-FD -> my_footprints:C_EEE-FT1V470AR
- J1: value PJ-063AH -> HC-DC-005-2.0M; footprint my_footprints:CUI_PJ-063AH -> easyeda2kicad:DC-IN-TH_DC-005-2.0
- J3: renamed from J4; value Screw_Terminal_01x04 -> Screw_Terminal_01x05
- R24, R25: footprint Resistor_SMD:R_0805_2012Metric -> Resistor_SMD:R_1206_3216Metric
- R3, R5, R6: footprint Resistor_SMD:R_0805_2012Metric -> Resistor_SMD:R_0603_1608Metric
- U7, U8: value MCP3551 -> MCP3551-E/SN
- moved J1 2.71 mm to (102.3, 120.2), turned to 90 degrees
- moved C16 0.43 mm to (54.9, 117.0)
Routing:
- net GND: track 617.7 -> 632.1 mm, vias 56 -> 59
- net +15V: track 43.5 -> 42.7 mm
