File: hardware/mystat_circuit_board/kicad_files/power.kicad_sch (KiCad schematic)
At the start: 17 parts, among them J1 PJ-063AH, U2 LTM8045, U3 ADP7182AUJZ-R7, U4 ADP7118AUJZ-5.0-R7

Commit message: revert to KiCAD 10 state before attempting reed relay changes, to merge into master
Parts:
- C3: LCSC C193627 -> (none); Part Number EEEFT1V470AR -> EEE-FT1V470AR
- R2: LCSC C2684603 -> (none); Manufacturer Viking Tech -> Panasonic Electronic Components; Part Number ARG05BTC8871 -> ERA-6AEB8871V
- R3: LCSC C706252 -> (none); Manufacturer YAGEO -> Panasonic Electronic Components; Part Number RT0805BRD0788K7L -> ERJ-PB6B8872V
- R5: LCSC C2681629 -> (none); Manufacturer Viking Tech -> Panasonic Electronic Components; Part Number ARG05BTC2943N -> ERJ-PB6B2943V
- R6: LCSC C2083549 -> (none); Manufacturer TE Connectivity -> Panasonic Electronic Components; Part Number RQ73C2A174KBTD -> ERJ-PB6B1743V
- U2: LCSC C581193 -> (none); Part Number LTM8045IY#PBF -> LTM8045IY
- U3: LCSC C514358 -> (none)
- U4: LCSC C141943 -> (none)
Changed lines of the file:
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@@
 			)
 		)
-		(property "Part Number" "LTM8045IY#PBF"
-			(at 68.58 186.69 0)
-			(hide yes)
-			(show_name no)
-			(do_not_autoplace no)
-			(effects
-				(font
-					(size 1.27 1.27)
-				)
-			)
-		)
-		(property "LCSC" "C581193"
+		(property "Part Number" "LTM8045IY"
 			(at 68.58 186.69 0)
 			(hide yes)
@@
 			)
 		)
-		(property "LCSC" ""
-			(at 91.44 168.91 0)
-			(hide yes)
-			(show_name no)
-			(do_not_autoplace no)
-			(effects
-				(font
-					(size 1.27 1.27)
-				)
-			)
-		)
 		(pin "2"
 		)
@@
 			)
 		)
-		(property "LCSC" ""
-			(at 44.45 201.93 0)
-			(hide yes)
-			(show_name no)
-			(do_not_autoplace no)
-			(effects
-				(font
-					(size 1.27 1.27)
-				)
-			)
-		)
 		(pin "1"
 		)
@@
 			)
 		)
-		(property "LCSC" ""
-			(at 44.45 215.9 0)
-			(hide yes)
-			(show_name no)
-			(do_not_autoplace no)
-			(effects
-				(font
-					(size 1.27 1.27)
-				)
-			)
-		)
 		(pin "1"
 		)
@@
 			)
 		)
-		(property "LCSC" ""
-			(at 44.45 167.64 0)
-			(hide yes)
-			(show_name no)
-			(do_not_autoplace no)
-			(effects
-				(font
-					(size 1.27 1.27)
-				)
-			)
-		)
 		(pin "1"
 		)
@@
 			)
 		)
-		(property "Part Number" "EEEFT1V470AR"
-			(at 77.47 96.52 0)
-			(hide yes)
-			(show_name no)
-			(do_not_autoplace no)
-			(effects
-				(font
-					(size 1.27 1.27)
-				)
-			)
-		)
-		(property "LCSC" "C193627"
+		(property "Part Number" "EEE-FT1V470AR"
 			(at 77.47 96.52 0)
 			(hide yes)
@@
 			)
 		)
-		(property "LCSC" "C141943"
-			(at 156.21 190.5 0)
-			(hide yes)
-			(show_name no)
-			(do_not_autoplace no)
-			(effects
-				(font
-					(size 1.27 1.27)
-				)
-			)
-		)
 		(pin "2"
 		)
@@
 			)
 		)
-		(property "LCSC" ""
-			(at 142.24 177.8 0)
-			(hide yes)
-			(show_name no)
-			(do_not_autoplace no)
-			(effects
-				(font
-					(size 1.27 1.27)
-				)
-			)
-		)
 		(pin "1"
 		)
@@
 			)
 		)
-		(property "LCSC" ""
-			(at 175.26 177.8 0)
-			(hide yes)
-			(show_name no)
-			(do_not_autoplace no)
-			(effects
-				(font
-					(size 1.27 1.27)
-				)
-			)
-		)
 		(pin "1"
 		)
@@
 			)
 		)
-		(property "Datasheet" "https://jlcpcb.com/api/file/downloadByFileSystemAccessId/8590167819447787521"
+		(property "Datasheet" "https://industrial.panasonic.com/cdbs/www-data/pdf/RDM0000/AOA0000C328.pdf"
 			(at 175.26 191.77 0)
 			(hide yes)
@@
 			)
 		)
-		(property "Manufacturer" "Viking Tech"
+		(property "Manufacturer" "Panasonic Electronic Components"
 			(at 175.26 191.77 0)
 			(hide yes)
@@
 			)
 		)
-		(property "Part Number" "ARG05BTC2943N"
-			(at 175.26 191.77 0)
-			(hide yes)
-			(show_name no)
-			(do_not_autoplace no)
-			(effects
-				(font
-					(size 1.27 1.27)
-				)
-			)
-		)
-		(property "LCSC" "C2681629"
+		(property "Part Number" "ERJ-PB6B2943V"
 			(at 175.26 191.77 0)
 			(hide yes)
@@
 			)
 		)
-		(property "Datasheet" "https://jlcpcb.com/api/file/downloadByFileSystemAccessId/8589819104925687808"
+		(property "Datasheet" "https://industrial.panasonic.com/cdbs/www-data/pdf/RDM0000/AOA0000C328.pdf"
 			(at 175.26 199.39 0)
 			(hide yes)
@@
 			)
 		)
-		(property "Manufacturer" "TE Connectivity"
+		(property "Manufacturer" "Panasonic Electronic Components"
 			(at 175.26 199.39 0)
 			(hide yes)
@@
 			)
 		)
-		(property "Part Number" "RQ73C2A174KBTD"
-			(at 175.26 199.39 0)
-			(hide yes)
-			(show_name no)
-			(do_not_autoplace no)
-			(effects
-				(font
-					(size 1.27 1.27)
-				)
-			)
-		)
-		(property "LCSC" "C2083549"
+		(property "Part Number" "ERJ-PB6B1743V"
 			(at 175.26 199.39 0)
 			(hide yes)
@@
 			)
 		)
-		(property "LCSC" "C514358"
-			(at 153.67 95.25 0)
-			(hide yes)
-			(show_name no)
-			(do_not_autoplace no)
-			(effects
-				(font
-					(size 1.27 1.27)
-				)
-			)
-		)
 		(pin "5"
 		)
@@
 			)
 		)
-		(property "LCSC" ""
-			(at 139.7 74.93 0)
-			(hide yes)
-			(show_name no)
-			(do_not_autoplace no)
-			(effects
-				(font
-					(size 1.27 1.27)
-				)
-			)
-		)
 		(pin "1"
 		)
@@
 			)
 		)
-		(property "LCSC" ""
-			(at 167.64 74.93 0)
-			(hide yes)
-			(show_name no)
-			(do_not_autoplace no)
-			(effects
-				(font
-					(size 1.27 1.27)
-				)
-			)
-		)
 		(pin "1"
 		)
@@
 			)
 		)
-		(property "Datasheet" "https://jlcpcb.com/api/file/downloadByFileSystemAccessId/8590171533386674176"
+		(property "Datasheet" "https://industrial.panasonic.com/cdbs/www-data/pdf/RDM0000/AOA0000C307.pdf"
 			(at 181.61 74.93 0)
 			(hide yes)
@@
 			)
 		)
-		(property "Manufacturer" "Viking Tech"
+		(property "Manufacturer" "Panasonic Electronic Components"
 			(at 181.61 74.93 0)
 			(hide yes)
@@
 			)
 		)
-		(property "Part Number" "ARG05BTC8871"
-			(at 181.61 74.93 0)
-			(hide yes)
-			(show_name no)
-			(do_not_autoplace no)
-			(effects
-				(font
-					(size 1.27 1.27)
-				)
-			)
-		)
-		(property "LCSC" "C2684603"
+		(property "Part Number" "ERA-6AEB8871V"
 			(at 181.61 74.93 0)
 			(hide yes)
@@
 			)
 		)
-		(property "Datasheet" "https://jlcpcb.com/api/file/downloadByFileSystemAccessId/8588935971161182208"
+		(property "Datasheet" "https://industrial.panasonic.com/cdbs/www-data/pdf/RDM0000/AOA0000C328.pdf"
 			(at 181.61 85.09 0)
 			(hide yes)
@@
 			)
 		)
-		(property "Manufacturer" "YAGEO"
+		(property "Manufacturer" "Panasonic Electronic Components"
 			(at 181.61 85.09 0)
 			(hide yes)
@@
 			)
 		)
-		(property "Part Number" "RT0805BRD0788K7L"
-			(at 181.61 85.09 0)
-			(hide yes)
-			(show_name no)
-			(do_not_autoplace no)
-			(effects
-				(font
-					(size 1.27 1.27)
-				)
-			)
-		)
-		(property "LCSC" "C706252"
+		(property "Part Number" "ERJ-PB6B8872V"
 			(at 181.61 85.09 0)
 			(hide yes)
@@
 			)
 		)
-		(property "LCSC" ""
-			(at 54.61 91.44 0)
-			(hide yes)
-			(show_name no)
-			(do_not_autoplace no)
-			(effects
-				(font
-					(size 1.27 1.27)
-				)
-			)
-		)

Commit message: merged Daniel's changes in to GUI. getting things ready in KiCAD 10 and finding substitute parts
Parts:
- C3: LCSC (none) -> C193627; Part Number EEE-FT1V470AR -> EEEFT1V470AR
- R2: LCSC (none) -> C2684603; Manufacturer Panasonic Electronic Components -> Viking Tech; Part Number ERA-6AEB8871V -> ARG05BTC8871
- R3: LCSC (none) -> C706252; Manufacturer Panasonic Electronic Components -> YAGEO; Part Number ERJ-PB6B8872V -> RT0805BRD0788K7L
- R5: LCSC (none) -> C2681629; Manufacturer Panasonic Electronic Components -> Viking Tech; Part Number ERJ-PB6B2943V -> ARG05BTC2943N
- R6: LCSC (none) -> C2083549; Manufacturer Panasonic Electronic Components -> TE Connectivity; Part Number ERJ-PB6B1743V -> RQ73C2A174KBTD
- U2: LCSC (none) -> C581193; Part Number LTM8045IY -> LTM8045IY#PBF
- U3: LCSC (none) -> C514358
- U4: LCSC (none) -> C141943
Changed lines of the file:
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@@
 			)
 		)
-		(property "Part Number" "LTM8045IY"
+		(property "Part Number" "LTM8045IY#PBF"
+			(at 68.58 186.69 0)
+			(hide yes)
+			(show_name no)
+			(do_not_autoplace no)
+			(effects
+				(font
+					(size 1.27 1.27)
+				)
+			)
+		)
+		(property "LCSC" "C581193"
 			(at 68.58 186.69 0)
 			(hide yes)
@@
 			)
 		)
+		(property "LCSC" ""
+			(at 91.44 168.91 0)
+			(hide yes)
+			(show_name no)
+			(do_not_autoplace no)
+			(effects
+				(font
+					(size 1.27 1.27)
+				)
+			)
+		)
 		(pin "2"
 		)
@@
 			)
 		)
+		(property "LCSC" ""
+			(at 44.45 201.93 0)
+			(hide yes)
+			(show_name no)
+			(do_not_autoplace no)
+			(effects
+				(font
+					(size 1.27 1.27)
+				)
+			)
+		)
 		(pin "1"
 		)
@@
 			)
 		)
+		(property "LCSC" ""
+			(at 44.45 215.9 0)
+			(hide yes)
+			(show_name no)
+			(do_not_autoplace no)
+			(effects
+				(font
+					(size 1.27 1.27)
+				)
+			)
+		)
 		(pin "1"
 		)
@@
 			)
 		)
+		(property "LCSC" ""
+			(at 44.45 167.64 0)
+			(hide yes)
+			(show_name no)
+			(do_not_autoplace no)
+			(effects
+				(font
+					(size 1.27 1.27)
+				)
+			)
+		)
 		(pin "1"
 		)
@@
 			)
 		)
-		(property "Part Number" "EEE-FT1V470AR"
+		(property "Part Number" "EEEFT1V470AR"
+			(at 77.47 96.52 0)
+			(hide yes)
+			(show_name no)
+			(do_not_autoplace no)
+			(effects
+				(font
+					(size 1.27 1.27)
+				)
+			)
+		)
+		(property "LCSC" "C193627"
 			(at 77.47 96.52 0)
 			(hide yes)
@@
 			)
 		)
+		(property "LCSC" "C141943"
+			(at 156.21 190.5 0)
+			(hide yes)
+			(show_name no)
+			(do_not_autoplace no)
+			(effects
+				(font
+					(size 1.27 1.27)
+				)
+			)
+		)
 		(pin "2"
 		)
@@
 			)
 		)
+		(property "LCSC" ""
+			(at 142.24 177.8 0)
+			(hide yes)
+			(show_name no)
+			(do_not_autoplace no)
+			(effects
+				(font
+					(size 1.27 1.27)
+				)
+			)
+		)
 		(pin "1"
 		)
@@
 			)
 		)
+		(property "LCSC" ""
+			(at 175.26 177.8 0)
+			(hide yes)
+			(show_name no)
+			(do_not_autoplace no)
+			(effects
+				(font
+					(size 1.27 1.27)
+				)
+			)
+		)
 		(pin "1"
 		)
@@
 			)
 		)
-		(property "Datasheet" "https://industrial.panasonic.com/cdbs/www-data/pdf/RDM0000/AOA0000C328.pdf"
+		(property "Datasheet" "https://jlcpcb.com/api/file/downloadByFileSystemAccessId/8590167819447787521"
 			(at 175.26 191.77 0)
 			(hide yes)
@@
 			)
 		)
-		(property "Manufacturer" "Panasonic Electronic Components"
+		(property "Manufacturer" "Viking Tech"
 			(at 175.26 191.77 0)
 			(hide yes)
@@
 			)
 		)
-		(property "Part Number" "ERJ-PB6B2943V"
+		(property "Part Number" "ARG05BTC2943N"
+			(at 175.26 191.77 0)
+			(hide yes)
+			(show_name no)
+			(do_not_autoplace no)
+			(effects
+				(font
+					(size 1.27 1.27)
+				)
+			)
+		)
+		(property "LCSC" "C2681629"
 			(at 175.26 191.77 0)
 			(hide yes)
@@
 			)
 		)
-		(property "Datasheet" "https://industrial.panasonic.com/cdbs/www-data/pdf/RDM0000/AOA0000C328.pdf"
+		(property "Datasheet" "https://jlcpcb.com/api/file/downloadByFileSystemAccessId/8589819104925687808"
 			(at 175.26 199.39 0)
 			(hide yes)
@@
 			)
 		)
-		(property "Manufacturer" "Panasonic Electronic Components"
+		(property "Manufacturer" "TE Connectivity"
 			(at 175.26 199.39 0)
 			(hide yes)
@@
 			)
 		)
-		(property "Part Number" "ERJ-PB6B1743V"
+		(property "Part Number" "RQ73C2A174KBTD"
+			(at 175.26 199.39 0)
+			(hide yes)
+			(show_name no)
+			(do_not_autoplace no)
+			(effects
+				(font
+					(size 1.27 1.27)
+				)
+			)
+		)
+		(property "LCSC" "C2083549"
 			(at 175.26 199.39 0)
 			(hide yes)
@@
 			)
 		)
+		(property "LCSC" "C514358"
+			(at 153.67 95.25 0)
+			(hide yes)
+			(show_name no)
+			(do_not_autoplace no)
+			(effects
+				(font
+					(size 1.27 1.27)
+				)
+			)
+		)
 		(pin "5"
 		)
@@
 			)
 		)
+		(property "LCSC" ""
+			(at 139.7 74.93 0)
+			(hide yes)
+			(show_name no)
+			(do_not_autoplace no)
+			(effects
+				(font
+					(size 1.27 1.27)
+				)
+			)
+		)
 		(pin "1"
 		)
@@
 			)
 		)
+		(property "LCSC" ""
+			(at 167.64 74.93 0)
+			(hide yes)
+			(show_name no)
+			(do_not_autoplace no)
+			(effects
+				(font
+					(size 1.27 1.27)
+				)
+			)
+		)
 		(pin "1"
 		)
@@
 			)
 		)
-		(property "Datasheet" "https://industrial.panasonic.com/cdbs/www-data/pdf/RDM0000/AOA0000C307.pdf"
+		(property "Datasheet" "https://jlcpcb.com/api/file/downloadByFileSystemAccessId/8590171533386674176"
 			(at 181.61 74.93 0)
 			(hide yes)
@@
 			)
 		)
-		(property "Manufacturer" "Panasonic Electronic Components"
+		(property "Manufacturer" "Viking Tech"
 			(at 181.61 74.93 0)
 			(hide yes)
@@
 			)
 		)
-		(property "Part Number" "ERA-6AEB8871V"
+		(property "Part Number" "ARG05BTC8871"
+			(at 181.61 74.93 0)
+			(hide yes)
+			(show_name no)
+			(do_not_autoplace no)
+			(effects
+				(font
+					(size 1.27 1.27)
+				)
+			)
+		)
+		(property "LCSC" "C2684603"
 			(at 181.61 74.93 0)
 			(hide yes)
@@
 			)
 		)
-		(property "Datasheet" "https://industrial.panasonic.com/cdbs/www-data/pdf/RDM0000/AOA0000C328.pdf"
+		(property "Datasheet" "https://jlcpcb.com/api/file/downloadByFileSystemAccessId/8588935971161182208"
 			(at 181.61 85.09 0)
 			(hide yes)
@@
 			)
 		)
-		(property "Manufacturer" "Panasonic Electronic Components"
+		(property "Manufacturer" "YAGEO"
 			(at 181.61 85.09 0)
 			(hide yes)
@@
 			)
 		)
-		(property "Part Number" "ERJ-PB6B8872V"
+		(property "Part Number" "RT0805BRD0788K7L"
+			(at 181.61 85.09 0)
+			(hide yes)
+			(show_name no)
+			(do_not_autoplace no)
+			(effects
+				(font
+					(size 1.27 1.27)
+				)
+			)
+		)
+		(property "LCSC" "C706252"
 			(at 181.61 85.09 0)
 			(hide yes)
@@
 			)
 		)
+		(property "LCSC" ""
+			(at 54.61 91.44 0)
+			(hide yes)
+			(show_name no)
+			(do_not_autoplace no)
+			(effects
+				(font
+					(size 1.27 1.27)
+				)
+			)
+		)
