File: hardware/mystat_circuit_board/kicad_files/power.kicad_sch (KiCad schematic)
At the start: 17 parts, among them J1 PJ-063AH, U2 LTM8045, U3 ADP7182AUJZ-R7, U4 ADP7118AUJZ-5.0-R7

Commit message: more pcb layout progress save
Parts:
- removed C3: 47 uF, my_footprints:EEE-FT1V470AR, symbol Device:C_Small
- added C3: 47 uF, easyeda2kicad:CAP-SMD_BD5.0-L5.3-W5.3-LS6.0-FD, symbol easyeda2kicad:EFVM035ADA470M0554
- C4, C7: MPN (none) -> CL31B475KBHNNNE
- C5, C6, C8, C9: MPN (none) -> C2012X7R1V475K125AC
- J1: MPN (none) -> PJ-063AH
- R1: MPN (none) -> ERJ-6ENF6042V
- R2: MPN (none) -> ERA-6AEB8871V
- R3: MPN (none) -> ERJ-PB6B8872V
- R4: MPN (none) -> ERJ-6ENF1783V
- R5: MPN (none) -> ERJ-PB6B2943V
- R6: MPN (none) -> ERJ-PB6B1743V
- U2: MPN (none) -> LTM8045IY
- U3: MPN (none) -> ADP7182AUJZ-R7
- U4: MPN (none) -> ADP7118AUJZ-5.0-R7
Connections:
- net +15V: now also C3.1
- net GND: now also C3.2

Commit message: mostly resistor changes
Parts:
- removed J1: PJ-063AH, my_footprints:CUI_PJ-063AH, symbol mylib:PJ-063AH
- added J1: HC-DC-005-2.0M, easyeda2kicad:DC-IN-TH_DC-005-2.0, symbol easyeda2kicad:HC-DC-005-2.0M
- C3: footprint easyeda2kicad:CAP-SMD_BD5.0-L5.3-W5.3-LS6.0-FD -> my_footprints:C_EEE-FT1V470AR; symbol easyeda2kicad:EFVM035ADA470M0554 -> Device:C_Polarized; LCSC Part C22387982 -> C193627; MPN EFVM035ADA470M0554 -> EEE-FT1V470AR; Manufacturer FOLLON(富隆电子) -> Panasonic Electronic Components; Part Number EFVM035ADA470M0554 -> (none)
- C4, C7: LCSC Part (none) -> C51205; Part Number CL31B475KBHNNNE -> (none)
- C5, C6, C8, C9: LCSC Part (none) -> C1779; MPN C2012X7R1V475K125AC -> CL21A475KAQNNNE; Manufacturer TDK Corporation -> Samsung Electro-Mechanics; Part Number C2012X7R1V475K125AC -> (none)
- R1: LCSC Part (none) -> C273994; MPN ERJ-6ENF6042V -> RC0805FR-0760K4L; Manufacturer Panasonic Electronic Components -> YAGEO; Part Number ERJ-6ENF6042V -> (none)
- R2: LCSC Part (none) -> C2684603; MPN ERA-6AEB8871V -> ARG05BTC8871; Manufacturer Panasonic Electronic Components -> Viking Tech; Part Number ERA-6AEB8871V -> (none)
- R3: footprint Resistor_SMD:R_0805_2012Metric -> Resistor_SMD:R_0603_1608Metric; LCSC Part (none) -> C728599; MPN ERJ-PB6B8872V -> RT0603BRD0788K7L; Manufacturer Panasonic Electronic Components -> YAGEO; Part Number ERJ-PB6B8872V -> (none)
- R4: LCSC Part (none) -> C228342; MPN ERJ-6ENF1783V -> AC0805FR-07178KL; Manufacturer Panasonic Electronic Components -> YAGEO; Part Number ERJ-6ENF1783V -> (none)
- R5: footprint Resistor_SMD:R_0805_2012Metric -> Resistor_SMD:R_0603_1608Metric; LCSC Part (none) -> C861286; MPN ERJ-PB6B2943V -> RT0603BRD07294KL; Manufacturer Panasonic Electronic Components -> YAGEO; Part Number ERJ-PB6B2943V -> (none)
- R6: footprint Resistor_SMD:R_0805_2012Metric -> Resistor_SMD:R_0603_1608Metric; LCSC Part (none) -> C1870358; MPN ERJ-PB6B1743V -> TNPW0603174KBEEA; Manufacturer Panasonic Electronic Components -> Vishay Intertec; Part Number ERJ-PB6B1743V -> (none)
- U2: LCSC Part (none) -> C581193; Part Number LTM8045IY -> (none)
- U3: LCSC Part (none) -> C514358; Part Number ADP7182AUJZ-R7 -> (none)
- U4: LCSC Part (none) -> C141943; Part Number ADP7118AUJZ-5.0-R7 -> (none)
Connections:
- net +15V: now also J1.5
- net GND: now also J1.3, J1.4
