File: hardware/mystat_circuit_board/kicad_files/analog.kicad_sch (KiCad schematic)
At the start: 46 parts, among them J3 SJ1-42534-SMT, K1 9011-05-11, K2 9011-05-11, K3 9011-05-11, K4 9011-05-11, K5 9011-05-11, U10 OPA192, U11 BUF634A, U12 ADG1419, U13 OPA192, U14 OPA192, U15 OPA192, U16 OPA192, U17 OPA192

Commit message: schematic: change electrode connections to screw terminals, BUF634A to HSOIC version with thermal pad
Parts:
- removed J3: SJ1-42534-SMT, my_footprints:CUI_SJ1-42534-SMT, symbol mylib:SJ1-42534-SMT
- removed U11: BUF634A, my_footprints:SOIC-8, symbol mylib:BUF634A
- added J4: Screw_Terminal_01x04, symbol Connector:Screw_Terminal_01x04
- added U11: BUF634AIDDAR, Package_SO:TI_SO-PowerPAD-8_ThermalVias, symbol Amplifier_Buffer:BUF634AxDDA
Connections:
- net +13.4V: now also U11.7 (V+)
- net -13.4V: now also U11.9 (THPAD)
- net CE: now also J4.4 (Pin_4)
- net RE: now also J4.2 (Pin_2)
- net SE: now also J4.3 (Pin_3)
- net WE: now also J4.1 (Pin_1)
- net at C24.1, K1.1, R10.1: now also U11.6
- net at U10.1: now also U11.3 (V_{IN})
Other:
- note added: "External connection to cell"
- note removed: "Jack for external connection to cell"
- moved on the sheet: C23, C24, C26, R11, U10
